Commit message: Add URDF links and joints for front and back wheels; remove unused STL files

File: ros_ws/src/pickeycar_description/urdf/pickeycar.urdf (robot description, URDF)
Before this commit: robot pickeycar, 17 links, 16 joints
Links:
- added link back_left_wheel, mass 0.0515309299357028; collision mesh filename=package://pickeycar_description/meshes/X3plus/visual/back_l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; visual mesh filename=package://pickeycar_description/meshes/X3plus/visual/back_l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
- added link back_right_wheel, mass 0.051540174053366; collision mesh filename=package://pickeycar_description/meshes/X3plus/visual/back_r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; visual mesh filename=package://pickeycar_description/meshes/X3plus/visual/back_r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
- added link front_left_wheel, mass 0.051543; collision mesh filename=package://pickeycar_description/meshes/X3plus/visual/front_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; visual mesh filename=package://pickeycar_description/meshes/X3plus/visual/front_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
- added link front_right_wheel, mass 0.051532; collision mesh filename=package://pickeycar_description/meshes/X3plus/visual/front_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; visual mesh filename=package://pickeycar_description/meshes/X3plus/visual/front_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
Joints:
- added joint back_left_joint: type continuous, parent base_link, child back_left_wheel, origin xyz=-0.115 0.105 -0.03954 rpy=1.5703 0 0, axis 0 0 1, limit effort=100 velocity=1
- added joint back_right_joint: type continuous, parent base_link, child back_right_wheel, origin xyz=-0.115 -0.105 -0.03946 rpy=-1.57 0 3.14159, axis 0 0 1, limit effort=100 velocity=1
- added joint front_left_joint: type continuous, parent base_link, child front_left_wheel, origin xyz=0.105 0.105 -0.0389 rpy=1.5703 0 0, axis 0 0 1, limit effort=100 velocity=1
- added joint front_right_joint: type continuous, parent base_link, child front_right_wheel, origin xyz=0.105 -0.105 -0.0389 rpy=-1.5703 0 0, axis 0 0 1, limit effort=100 velocity=1
